Commit message: initial iris-modquad frame

File: big_modquad/config/rotors_description/urdf/iris.xacro (robot description, xacro)
@@ -7,4 +7,5 @@
   <xacro:property name="mesh_scale" value="1 1 1"/>
   <xacro:property name="mesh_scale_prop" value="1 1 1"/>
+  <xacro:property name="mesh_scale_guard" value="0.0025 0.0025 0.0025"/>
   <xacro:property name="mass" value="1.5" /> <!-- [kg] -->
   <xacro:property name="body_width" value="0.47" /> <!-- [m] -->
@@ -32,4 +33,7 @@
     <inertia ixx="0.0347563" ixy="0.0" ixz="0.0" iyy="0.0458929" iyz="0.0" izz="0.0977" /> <!-- [kg.m^2] [kg.m^2] [kg.m^2] [kg.m^2] [kg.m^2] [kg.m^2] -->
   </xacro:property>
+  <xacro:property name="prop_guard_inertia">
+    <inertia ixx="0.009" ixy="0.0" ixz="0.0" iyy="0.00458929" iyz="0.0" izz="0.00977" /> <!-- [kg.m^2] [kg.m^2] [kg.m^2] [kg.m^2] [kg.m^2] [kg.m^2] -->
+  </xacro:property>
   <!-- inertia of a single rotor, assuming it is a cuboid. Height=3mm, width=15mm -->
   <xacro:property name="rotor_inertia">
@@ -54,4 +58,13 @@
     <xacro:insert_block name="body_inertia" />
   </xacro:multirotor_base_macro>
+  <xacro:prop_guard_macro
+    robot_namespace="${namespace}"
+    mass="0.07"
+    body_width="${body_width + 0.08}"
+    body_height="${body_height + 0.06}"
+    mesh_scale="${mesh_scale_guard}"
+    >
+    <xacro:insert_block name="prop_guard_inertia" />
+  </xacro:prop_guard_macro>
   <!-- Instantiate rotors -->
   <xacro:vertical_rotor

File: big_modquad/config/rotors_description/urdf/iris_base.xacro (robot description, xacro)
@@ -84,5 +84,5 @@
     >
     <box size="0.01 0.01 0.01" />
-    <origin xyz="0.1 0.0 0.0" rpy="0.0 0.0 0.0" />
+    <origin xyz="0.15 0.0 0.05" rpy="0.0 0.0 0.0" />
   </xacro:camera_macro>
   <xacro:if value="$(arg enable_mavlink_interface)">

File: big_modquad/config/rotors_description/urdf/multirotor_base.xacro (robot description, xacro)
@@ -58,4 +58,48 @@
       <material>Gazebo/${color}</material>
       <collision name='base_link_inertia_collision'>
+        <surface>
+          <contact>
+            <ode>
+              <min_depth>0.001</min_depth>
+              <max_vel>0.0</max_vel>
+            </ode>
+          </contact>
+          <friction>
+            <ode/>
+          </friction>
+        </surface>
+      </collision>
+   </gazebo>
+  </xacro:macro>
+  <xacro:macro name="prop_guard_macro"
+    params="robot_namespace mass body_width body_height mesh_scale *inertia">
+    <joint name="prop_guard_${robot_namespace}_joint" type="fixed">
+      <origin xyz="0 0 0" rpy="0 0 0" />
+      <parent link="base_link" />
+      <child link="prop_guard_${robot_namespace}" />
+    </joint>
+    <link name="prop_guard_${robot_namespace}">
+      <inertial>
+        <mass value="${mass}" />
+        <origin xyz="0 0 0" />
+        <xacro:insert_block name="inertia" />
+      </inertial>
+      <visual>
+        <origin xyz="0.27 -0.29 -0.22" rpy="1.57079632679 0 3.14159265359" />
+        <geometry>
+          <mesh filename="package://rotors_description/meshes/TMotorAssembly.STL"
+            scale="${mesh_scale}" />
+        </geometry>
+      </visual>
+      <collision>
+        <origin xyz="0 0 0" rpy="0 0 0" />
+        <geometry>
+          <box size="${body_width} ${body_width} ${body_height}" />
+        </geometry>
+      </collision>
+    </link>
+    <gazebo reference="prop_guard_${robot_namespace}">
+      <material>Gazebo/DarkGrey</material>
+      <collision name='prop_guard_${robot_namespace}_inertia_collision'>
         <surface>
           <contact>
