Commit message: added whycon tags and frame

File: big_modquad/config/rotors_description/urdf/component_snippets.xacro (robot description, xacro)
@@ -103,4 +103,34 @@
         </plugin>
       </sensor>
+    </gazebo>
+  </xacro:macro>
+  <xacro:macro name="tag_mount_macro" params="namespace suffix *cylinder *origin">
+    <link name="${namespace}/${suffix}_tag_mount_link">
+      <collision>
+        <origin xyz="0 0 0" rpy="0 0 0" />
+        <geometry>
+          <xacro:insert_block name="cylinder" />
+        </geometry>
+      </collision>
+        <visual>
+          <origin xyz="0 0 0" rpy="0 1.57079632679 0" />
+          <geometry>
+            <xacro:insert_block name="cylinder" />
+          </geometry>
+          <material name="red" />
+        </visual>
+      <inertial>
+        <mass value="1e-5" />
+        <origin xyz="0 0 0" rpy="0 0 0" />
+        <inertia ixx="1e-6" ixy="0" ixz="0" iyy="1e-6" iyz="0" izz="1e-6" />
+      </inertial>
+    </link>
+    <joint name="${namespace}/${suffix}_tag_mount_joint" type="fixed">
+      <xacro:insert_block name="origin" />
+      <parent link="base_link" />
+      <child link="${namespace}/${suffix}_tag_mount_link" />
+    </joint>
+    <gazebo reference="${namespace}/${suffix}_tag_mount_link">
+      <material>whycon</material>
     </gazebo>
   </xacro:macro>

File: big_modquad/config/rotors_description/urdf/iris_base.xacro (robot description, xacro)
@@ -68,4 +68,25 @@
     >
   </xacro:barometer_plugin_macro>
+  <xacro:tag_mount_macro
+    namespace="${namespace}"
+    suffix="back"
+    >
+    <box size="0.14 0.14 0.001" />
+    <origin xyz="-0.265 0 0.05" rpy="0 0 0" />
+  </xacro:tag_mount_macro>
+  <xacro:tag_mount_macro
+    namespace="${namespace}"
+    suffix="right"
+    >
+    <box size="0.14 0.14 0.001" />
+    <origin xyz="0 -0.265 0.05" rpy="0 0 1.57079632679" />
+  </xacro:tag_mount_macro>
+  <xacro:tag_mount_macro
+    namespace="${namespace}"
+    suffix="left"
+    >
+    <box size="0.14 0.14 0.001" />
+    <origin xyz="0 0.27 0.05" rpy="0 0 1.57079632679" />
+  </xacro:tag_mount_macro>
   <xacro:camera_macro
     namespace="${namespace}"

File: big_modquad/config/rotors_description/urdf/multirotor_base.xacro (robot description, xacro)
@@ -100,5 +100,6 @@
     </link>
     <gazebo reference="prop_guard_${robot_namespace}">
-      <material>Gazebo/DarkGrey</material>
+      <material>whycon</material>
+      <!--material>Gazebo/DarkGrey</material-->
       <collision name='prop_guard_${robot_namespace}_inertia_collision'>
         <surface>

Commit message: integrated magnets into build

File: big_modquad/config/rotors_description/urdf/component_snippets.xacro (robot description, xacro)
@@ -103,4 +103,44 @@
         </plugin>
       </sensor>
+    </gazebo>
+  </xacro:macro>
+  <xacro:macro name="magnet_plugin_macro"
+    params="namespace suffix should_publish strength *origin">
+    <link name="${namespace}/magnet_${suffix}_link">
+      <collision>
+        <origin xyz="0 0 0" rpy="0 0 0" />
+        <geometry>
+          <box size="0.0015 0.017 0.017" />
+        </geometry>
+      </collision>
+      <visual>
+        <origin xyz="0 0 0" rpy="0 0 0" />
+        <geometry>
+          <box size="0.0015 0.017 0.017" />
+        </geometry>
+        <material name="red" />
+      </visual>
+      <inertial>
+        <mass value="1e-6" />
+        <origin xyz="0 0 0" rpy="0 0 0" />
+        <inertia ixx="1e-9" ixy="0" ixz="0" iyy="1e-9" iyz="0" izz="1e-9" />
+      </inertial>
+    </link>
+    <joint name="${namespace}/magnet_${suffix}_joint" type="fixed">
+      <xacro:insert_block name="origin" />
+      <parent link="base_link" />
+      <child link="${namespace}/magnet_${suffix}_link" />
+    </joint>
+    <gazebo>
+      <plugin filename="libgazebo_dipole_magnet.so" name="magnet_plugin">
+        <dipole_moment>${strength}</dipole_moment>
+        <shouldPublish>${should_publish}</shouldPublish>
+        <robotNamespace>${namespace}</robotNamespace>
+        <bodyName>${namespace}/magnet_${suffix}_link</bodyName>
+        <topicNs>${namespace}/magnet_${suffix}_link</topicNs>
+      </plugin>
+    </gazebo>
+    <gazebo reference="${namespace}/magnet_${suffix}_link">
+      <material>Gazebo/DarkGrey</material>
     </gazebo>
   </xacro:macro>

File: big_modquad/config/rotors_description/urdf/iris_base.xacro (robot description, xacro)
@@ -68,4 +68,12 @@
     >
   </xacro:barometer_plugin_macro>
+  <xacro:magnet_plugin_macro
+    namespace="${namespace}"
+    suffix="1"
+    strength="0 0 1.5"
+    should_publish="true"
+    >
+    <origin xyz="-0.965 0 0.05" rpy="0 0 0" />
+  </xacro:magnet_plugin_macro>
   <xacro:tag_mount_macro
     namespace="${namespace}"

Commit message: fron and back magnets working, left and right need work

File: big_modquad/config/rotors_description/urdf/component_snippets.xacro (robot description, xacro)
@@ -111,18 +111,20 @@
         <origin xyz="0 0 0" rpy="0 0 0" />
         <geometry>
-          <box size="0.0015 0.017 0.017" />
+          <!--box size="0.15 0.017 0.017" /-->
+          <cylinder length="0.0015" radius="0.0085" />
         </geometry>
       </collision>
       <visual>
-        <origin xyz="0 0 0" rpy="0 0 0" />
+        <origin xyz="0 0 0" rpy="0 1.57079632679 0" />
         <geometry>
-          <box size="0.0015 0.017 0.017" />
+          <!--box size="0.0015 0.017 0.017" /-->
+          <cylinder length="0.0015" radius="0.0085" />
         </geometry>
         <material name="red" />
       </visual>
       <inertial>
-        <mass value="1e-6" />
-        <origin xyz="0 0 0" rpy="0 0 0" />
-        <inertia ixx="1e-9" ixy="0" ixz="0" iyy="1e-9" iyz="0" izz="1e-9" />
+        <mass value="1e-3" />
+        <origin xyz="0 0 0" rpy="0 0 0" />
+        <inertia ixx="1e-6" ixy="0" ixz="0" iyy="1e-6" iyz="0" izz="1e-9" />
       </inertial>
     </link>

File: big_modquad/config/rotors_description/urdf/iris.xacro (robot description, xacro)
@@ -61,6 +61,6 @@
     robot_namespace="${namespace}"
     mass="0.07"
-    body_width="${body_width + 0.08}"
-    body_height="${body_height + 0.06}"
+    body_width="${body_width-0.02}"
+    body_height="${body_height}"
     mesh_scale="${mesh_scale_guard}"
     >

File: big_modquad/config/rotors_description/urdf/iris_base.xacro (robot description, xacro)
@@ -68,11 +68,196 @@
     >
   </xacro:barometer_plugin_macro>
-  <xacro:magnet_plugin_macro
-    namespace="${namespace}"
-    suffix="1"
-    strength="0 0 1.5"
-    should_publish="true"
-    >
-    <origin xyz="-0.965 0 0.05" rpy="0 0 0" />
+  <!--xacro:magnet_plugin_macro
+    namespace="${namespace}"
+    suffix="1_back_left_forward"
+    strength="0 0 0.3"
+    should_publish="true"
+    >
+    <origin xyz="-0.277 0.135 -0.006" rpy="0 3.14159265359 0" />
+  </xacro:magnet_plugin_macro-->
+  <!--xacro:magnet_plugin_macro
+    namespace="${namespace}"
+    suffix="2_back_left_forward"
+    strength="0 0 0.3"
+    should_publish="true"
+    >
+    <origin xyz="-0.277 0.135 0.049" rpy="0 3.14159265359 0" />
+  </xacro:magnet_plugin_macro-->
+  <xacro:magnet_plugin_macro
+    namespace="${namespace}"
+    suffix="3_back_left_forward"
+    strength="0 0 0.3"
+    should_publish="true"
+    >
+    <origin xyz="-0.277 0.135 0.105" rpy="0 3.14159265359 0" />
+  </xacro:magnet_plugin_macro>
+  <!--xacro:magnet_plugin_macro
+    namespace="${namespace}"
+    suffix="1_back_right_backward"
+    strength="0 0 0.3"
+    should_publish="true"
+    >
+    <origin xyz="-0.277 -0.1263 -0.006" rpy="0 0 3.14159265359" />
+  </xacro:magnet_plugin_macro-->
+  <!--xacro:magnet_plugin_macro
+    namespace="${namespace}"
+    suffix="2_back_right_backward"
+    strength="0 0 0.3"
+    should_publish="true"
+    >
+    <origin xyz="-0.277 -0.1263 0.049" rpy="0 0 3.14159265359" />
+  </xacro:magnet_plugin_macro-->
+  <xacro:magnet_plugin_macro
+    namespace="${namespace}"
+    suffix="3_back_right_backward"
+    strength="0 0 0.3"
+    should_publish="true"
+    >
+    <origin xyz="-0.277 -0.1263 0.105" rpy="0 0 3.14159265359" />
+  </xacro:magnet_plugin_macro>
+  <!--xacro:magnet_plugin_macro
+    namespace="${namespace}"
+    suffix="4_front_right_forward"
+    strength="0 0 0.3"
+    should_publish="true"
+    >
+    <origin xyz="0.269 -0.1263 -0.006" rpy="0 3.14159265359 3.14159265359" />
+  </xacro:magnet_plugin_macro-->
+<!--pi=3.14159265359-->
+  <!--xacro:magnet_plugin_macro
+    namespace="${namespace}"
+    suffix="5_front_right_forward"
+    strength="0 0 2"
+    should_publish="true"
+    >
+    <origin xyz="0.269 -0.1263 0.049" rpy="0 3.14159265359 3.14159265359" />
+  </xacro:magnet_plugin_macro-->
+  <xacro:magnet_plugin_macro
+    namespace="${namespace}"
+    suffix="6_front_right_forward"
+    strength="0 0 0.3"
+    should_publish="true"
+    >
+    <origin xyz="0.269 -0.1263 0.105" rpy="0 3.14159265359 3.14159265359" />
+  </xacro:magnet_plugin_macro>
+  <!--xacro:magnet_plugin_macro
+    namespace="${namespace}"
+    suffix="4_front_left_backward"
+    strength="0 0 0.3"
+    should_publish="true"
+    >
+    <origin xyz="0.269 0.135 -0.006" rpy="0 0 0" />
+  </xacro:magnet_plugin_macro>
+  <xacro:magnet_plugin_macro
+    namespace="${namespace}"
+    suffix="5_front_left_backward"
+    strength="0 0 0.3"
+    should_publish="true"
+    >
+    <origin xyz="0.269 0.135 0.049" rpy="0 0 0" />
+  </xacro:magnet_plugin_macro-->
+  <xacro:magnet_plugin_macro
+    namespace="${namespace}"
+    suffix="6_front_left_backward"
+    strength="0 0 0.3"
+    should_publish="true"
+    >
+    <origin xyz="0.269 0.135 0.105" rpy="0 0 0" />
+  </xacro:magnet_plugin_macro>
+  <!--xacro:magnet_plugin_macro
+    namespace="${namespace}"
+    suffix="7_right_back_forward"
+    strength="0 0 0.4"
+    should_publish="true"
+    >
+    <origin xyz="-0.134 -0.269 -0.006" rpy="3.14159265359 0 1.57079632679" />
+  </xacro:magnet_plugin_macro>
+  <xacro:magnet_plugin_macro
+    namespace="${namespace}"
+    suffix="8_right_back_forward"
+    strength="0 0 0.4"
+    should_publish="true"
+    >
+    <origin xyz="-0.134 -0.269 0.049" rpy="3.14159265359 0 1.57079632679" />
+  </xacro:magnet_plugin_macro-->
+  <xacro:magnet_plugin_macro
+    namespace="${namespace}"
+    suffix="9_right_back_forward"
+    strength="0 0 0.4"
+    should_publish="true"
+    >
+    <origin xyz="-0.134 -0.269 0.105" rpy="3.14159265359 0 1.57079632679" />
+  </xacro:magnet_plugin_macro>
+  <!--xacro:magnet_plugin_macro
+    namespace="${namespace}"
+    suffix="7_right_front_backward"
+    strength="0 0 0.4"
+    should_publish="true"
+    >
+    <origin xyz="0.127 -0.269 -0.006" rpy="0 0 -1.57079632679" />
+  </xacro:magnet_plugin_macro>
+  <xacro:magnet_plugin_macro
+    namespace="${namespace}"
+    suffix="8_right_front_backward"
+    strength="0 0 0.4"
+    should_publish="true"
+    >
+    <origin xyz="0.127 -0.269 0.049" rpy="0 0 -1.57079632679" />
+  </xacro:magnet_plugin_macro-->
+  <xacro:magnet_plugin_macro
+    namespace="${namespace}"
+    suffix="9_right_front_backward"
+    strength="0 0 0.4"
+    should_publish="true"
+    >
+    <origin xyz="0.127 -0.269 0.105" rpy="0 0 -1.57079632679" />
+  </xacro:magnet_plugin_macro>
+  <!--xacro:magnet_plugin_macro
+    namespace="${namespace}"
+    suffix="10_left_front_forward"
+    strength="0 0 0.4"
+    should_publish="true"
+    >
+    <origin xyz="0.127 0.278 -0.006" rpy="0 0 -1.57079632679" />
+  </xacro:magnet_plugin_macro>
+  <xacro:magnet_plugin_macro
+    namespace="${namespace}"
+    suffix="11_left_front_forward"
+    strength="0 0 0.4"
+    should_publish="true"
+    >
+    <origin xyz="0.127 0.278 0.049" rpy="0 0 -1.57079632679" />
+  </xacro:magnet_plugin_macro-->
+  <xacro:magnet_plugin_macro
+    namespace="${namespace}"
+    suffix="12_left_front_forward"
+    strength="0 0 0.4"
+    should_publish="true"
+    >
+    <origin xyz="0.127 0.278 0.105" rpy="0 0 -1.57079632679" />
+  </xacro:magnet_plugin_macro>
+  <!--xacro:magnet_plugin_macro
+    namespace="${namespace}"
+    suffix="10_left_back_backward"
+    strength="0 0 0.4"
+    should_publish="true"
+    >
+    <origin xyz="-0.135 0.278 -0.006" rpy="0 0 1.57079632679" />
+  </xacro:magnet_plugin_macro>
+  <xacro:magnet_plugin_macro
+    namespace="${namespace}"
+    suffix="11_left_back_backward"
+    strength="0 0 0.4"
+    should_publish="true"
+    >
+    <origin xyz="-0.135 0.278 0.049" rpy="0 0 1.57079632679" />
+  </xacro:magnet_plugin_macro-->
+  <xacro:magnet_plugin_macro
+    namespace="${namespace}"
+    suffix="12_left_back_backward"
+    strength="0 0 0.4"
+    should_publish="true"
+    >
+    <origin xyz="-0.135 0.278 0.105" rpy="0 0 1.57079632679" />
   </xacro:magnet_plugin_macro>
   <xacro:tag_mount_macro
