Commit message: full quad sim build complete

File: big_modquad/config/rotors_description/urdf/component_snippets.xacro (robot description, xacro)
@@ -110,4 +110,5 @@
       <collision>
         <origin xyz="0 0 0" rpy="0 0 0" />
+        <!--xacro:insert_block name="origin" /-->
         <geometry>
           <!--box size="0.15 0.017 0.017" /-->
@@ -147,8 +148,35 @@
     </gazebo>
   </xacro:macro>
+  <xacro:macro name="magnet_guard_macro"
+    params="namespace suffix *origin">
+    <link name="${namespace}/magnet_guard_${suffix}_link">
+      <collision>
+        <origin xyz="0 0 0" rpy="0 0 0" />
+        <!--xacro:insert_block name="origin" /-->
+        <geometry>
+          <box size="0.01 0.04 0.15" />
+        </geometry>
+      </collision>
+      <visual>
+        <origin xyz="0 0 0" rpy="0 0 0" />
+        <geometry>
+          <box size="0.01 0.04 0.15" />
+        </geometry>
+      </visual>
+    </link>
+    <joint name="${namespace}/magnet_guard_${suffix}_joint" type="fixed">
+      <xacro:insert_block name="origin" />
+      <parent link="base_link" />
+      <child link="${namespace}/magnet_guard_${suffix}_link" />
+    </joint>
+    <gazebo reference="${namespace}/magnet_guard_${suffix}_link">
+      <material>Gazebo/TurquoiseGlow</material>
+    </gazebo>
+  </xacro:macro>
   <xacro:macro name="tag_mount_macro" params="namespace suffix *cylinder *origin">
     <link name="${namespace}/${suffix}_tag_mount_link">
       <collision>
         <origin xyz="0 0 0" rpy="0 0 0" />
+        <!--xacro:insert_block name="origin" /-->
         <geometry>
           <xacro:insert_block name="cylinder" />

File: big_modquad/config/rotors_description/urdf/iris.xacro (robot description, xacro)
@@ -6,5 +6,5 @@
   <xacro:property name="mesh_file" value="iris.stl" />
   <xacro:property name="mesh_scale" value="1 1 1"/>
-  <xacro:property name="mesh_scale_prop" value="1 1 1"/>
+  <xacro:property name="mesh_scale_prop" value="0.5 0.5 1"/>
   <xacro:property name="mesh_scale_guard" value="0.0025 0.0025 0.0025"/>
   <xacro:property name="mass" value="1.5" /> <!-- [kg] -->

File: big_modquad/config/rotors_description/urdf/iris_base.xacro (robot description, xacro)
@@ -68,81 +68,129 @@
     >
   </xacro:barometer_plugin_macro>
-  <!--xacro:magnet_plugin_macro
+  <xacro:magnet_guard_macro
+    namespace="${namespace}"
+    suffix="back_left"
+    >
+    <origin xyz="-0.282 0.135 0.048" rpy="0 0 0" />
+  </xacro:magnet_guard_macro>
+  <xacro:magnet_guard_macro
+    namespace="${namespace}"
+    suffix="back_right"
+    >
+    <origin xyz="-0.282 -0.1263 0.048" rpy="0 0 0" />
+  </xacro:magnet_guard_macro>
+  <xacro:magnet_guard_macro
+    namespace="${namespace}"
+    suffix="front_left"
+    >
+    <origin xyz="0.274 0.135 0.048" rpy="0 0 0" />
+  </xacro:magnet_guard_macro>
+  <xacro:magnet_guard_macro
+    namespace="${namespace}"
+    suffix="front_right"
+    >
+    <origin xyz="0.274 -0.1263 0.048" rpy="0 0 0" />
+  </xacro:magnet_guard_macro>
+  <xacro:magnet_guard_macro
+    namespace="${namespace}"
+    suffix="right_front"
+    >
+    <origin xyz="0.132 -0.269 0.048" rpy="0 0 1.57079632679" />
+  </xacro:magnet_guard_macro>
+  <xacro:magnet_guard_macro
+    namespace="${namespace}"
+    suffix="right_back"
+    >
+    <origin xyz="-0.139 -0.269 0.048" rpy="0 0 1.57079632679" />
+  </xacro:magnet_guard_macro>
+  <xacro:magnet_guard_macro
+    namespace="${namespace}"
+    suffix="left_front"
+    >
+    <origin xyz="0.132 0.278 0.048" rpy="0 0 1.57079632679" />
+  </xacro:magnet_guard_macro>
+  <xacro:magnet_guard_macro
+    namespace="${namespace}"
+    suffix="left_back"
+    >
+    <origin xyz="-0.14 0.278 0.048" rpy="0 0 1.57079632679" />
+  </xacro:magnet_guard_macro>
+  <xacro:magnet_plugin_macro
     namespace="${namespace}"
     suffix="1_back_left_forward"
-    strength="0 0 0.3"
+    strength="0 0 1"
     should_publish="true"
     >
     <origin xyz="-0.277 0.135 -0.006" rpy="0 3.14159265359 0" />
-  </xacro:magnet_plugin_macro-->
-  <!--xacro:magnet_plugin_macro
+  </xacro:magnet_plugin_macro>
+  <xacro:magnet_plugin_macro
     namespace="${namespace}"
     suffix="2_back_left_forward"
-    strength="0 0 0.3"
+    strength="0 0 1"
     should_publish="true"
     >
     <origin xyz="-0.277 0.135 0.049" rpy="0 3.14159265359 0" />
-  </xacro:magnet_plugin_macro-->
+  </xacro:magnet_plugin_macro>
   <xacro:magnet_plugin_macro
     namespace="${namespace}"
     suffix="3_back_left_forward"
-    strength="0 0 0.3"
+    strength="0 0 1"
     should_publish="true"
     >
     <origin xyz="-0.277 0.135 0.105" rpy="0 3.14159265359 0" />
   </xacro:magnet_plugin_macro>
-  <!--xacro:magnet_plugin_macro
+  <xacro:magnet_plugin_macro
     namespace="${namespace}"
     suffix="1_back_right_backward"
-    strength="0 0 0.3"
+    strength="0 0 1"
     should_publish="true"
     >
     <origin xyz="-0.277 -0.1263 -0.006" rpy="0 0 3.14159265359" />
-  </xacro:magnet_plugin_macro-->
-  <!--xacro:magnet_plugin_macro
+  </xacro:magnet_plugin_macro>
+  <xacro:magnet_plugin_macro
     namespace="${namespace}"
     suffix="2_back_right_backward"
-    strength="0 0 0.3"
+    strength="0 0 1"
     should_publish="true"
     >
     <origin xyz="-0.277 -0.1263 0.049" rpy="0 0 3.14159265359" />
-  </xacro:magnet_plugin_macro-->
+  </xacro:magnet_plugin_macro>
   <xacro:magnet_plugin_macro
     namespace="${namespace}"
     suffix="3_back_right_backward"
-    strength="0 0 0.3"
+    strength="0 0 1"
     should_publish="true"
     >
     <origin xyz="-0.277 -0.1263 0.105" rpy="0 0 3.14159265359" />
   </xacro:magnet_plugin_macro>
-  <!--xacro:magnet_plugin_macro
+  <xacro:magnet_plugin_macro
     namespace="${namespace}"
     suffix="4_front_right_forward"
-    strength="0 0 0.3"
+    strength="0 0 1"
     should_publish="true"
     >
     <origin xyz="0.269 -0.1263 -0.006" rpy="0 3.14159265359 3.14159265359" />
-  </xacro:magnet_plugin_macro-->
+  </xacro:magnet_plugin_macro>
 <!--pi=3.14159265359-->
-  <!--xacro:magnet_plugin_macro
+  <xacro:magnet_plugin_macro
     namespace="${namespace}"
     suffix="5_front_right_forward"
-    strength="0 0 2"
+    strength="0 0 1"
     should_publish="true"
     >
     <origin xyz="0.269 -0.1263 0.049" rpy="0 3.14159265359 3.14159265359" />
-  </xacro:magnet_plugin_macro-->
+  </xacro:magnet_plugin_macro>
   <xacro:magnet_plugin_macro
     namespace="${namespace}"
     suffix="6_front_right_forward"
-    strength="0 0 0.3"
+    strength="0 0 1"
     should_publish="true"
     >
     <origin xyz="0.269 -0.1263 0.105" rpy="0 3.14159265359 3.14159265359" />
   </xacro:magnet_plugin_macro>
-  <!--xacro:magnet_plugin_macro
+  <xacro:magnet_plugin_macro
     namespace="${namespace}"
     suffix="4_front_left_backward"
-    strength="0 0 0.3"
+    strength="0 0 1"
     should_publish="true"
     >
@@ -152,21 +200,21 @@
     namespace="${namespace}"
     suffix="5_front_left_backward"
-    strength="0 0 0.3"
+    strength="0 0 1"
     should_publish="true"
     >
     <origin xyz="0.269 0.135 0.049" rpy="0 0 0" />
-  </xacro:magnet_plugin_macro-->
+  </xacro:magnet_plugin_macro>
   <xacro:magnet_plugin_macro
     namespace="${namespace}"
     suffix="6_front_left_backward"
-    strength="0 0 0.3"
+    strength="0 0 1"
     should_publish="true"
     >
     <origin xyz="0.269 0.135 0.105" rpy="0 0 0" />
   </xacro:magnet_plugin_macro>
-  <!--xacro:magnet_plugin_macro
+  <xacro:magnet_plugin_macro
     namespace="${namespace}"
     suffix="7_right_back_forward"
-    strength="0 0 0.4"
+    strength="0 0 1"
     should_publish="true"
     >
@@ -176,21 +224,21 @@
     namespace="${namespace}"
     suffix="8_right_back_forward"
-    strength="0 0 0.4"
+    strength="0 0 1"
     should_publish="true"
     >
     <origin xyz="-0.134 -0.269 0.049" rpy="3.14159265359 0 1.57079632679" />
-  </xacro:magnet_plugin_macro-->
+  </xacro:magnet_plugin_macro>
   <xacro:magnet_plugin_macro
     namespace="${namespace}"
     suffix="9_right_back_forward"
-    strength="0 0 0.4"
+    strength="0 0 1"
     should_publish="true"
     >
     <origin xyz="-0.134 -0.269 0.105" rpy="3.14159265359 0 1.57079632679" />
   </xacro:magnet_plugin_macro>
-  <!--xacro:magnet_plugin_macro
+  <xacro:magnet_plugin_macro
     namespace="${namespace}"
     suffix="7_right_front_backward"
-    strength="0 0 0.4"
+    strength="0 0 1"
     should_publish="true"
     >
@@ -200,45 +248,45 @@
     namespace="${namespace}"
     suffix="8_right_front_backward"
-    strength="0 0 0.4"
+    strength="0 0 1"
     should_publish="true"
     >
     <origin xyz="0.127 -0.269 0.049" rpy="0 0 -1.57079632679" />
-  </xacro:magnet_plugin_macro-->
+  </xacro:magnet_plugin_macro>
   <xacro:magnet_plugin_macro
     namespace="${namespace}"
     suffix="9_right_front_backward"
-    strength="0 0 0.4"
+    strength="0 0 1"
     should_publish="true"
     >
     <origin xyz="0.127 -0.269 0.105" rpy="0 0 -1.57079632679" />
   </xacro:magnet_plugin_macro>
-  <!--xacro:magnet_plugin_macro
+  <xacro:magnet_plugin_macro
     namespace="${namespace}"
     suffix="10_left_front_forward"
-    strength="0 0 0.4"
-    should_publish="true"
-    >
-    <origin xyz="0.127 0.278 -0.006" rpy="0 0 -1.57079632679" />
+    strength="0 0 1"
+    should_publish="true"
+    >
+    <origin xyz="0.127 0.278 -0.006" rpy="3.14159265359  0 -1.57079632679" />
   </xacro:magnet_plugin_macro>
   <xacro:magnet_plugin_macro
     namespace="${namespace}"
     suffix="11_left_front_forward"
-    strength="0 0 0.4"
-    should_publish="true"
-    >
-    <origin xyz="0.127 0.278 0.049" rpy="0 0 -1.57079632679" />
-  </xacro:magnet_plugin_macro-->
+    strength="0 0 1"
+    should_publish="true"
+    >
+    <origin xyz="0.127 0.278 0.049" rpy="3.14159265359   0 -1.57079632679" />
+  </xacro:magnet_plugin_macro>
   <xacro:magnet_plugin_macro
     namespace="${namespace}"
     suffix="12_left_front_forward"
-    strength="0 0 0.4"
-    should_publish="true"
-    >
-    <origin xyz="0.127 0.278 0.105" rpy="0 0 -1.57079632679" />
-  </xacro:magnet_plugin_macro>
-  <!--xacro:magnet_plugin_macro
+    strength="0 0 1"
+    should_publish="true"
+    >
+    <origin xyz="0.127 0.278 0.105" rpy="3.14159265359 0 -1.57079632679" />
+  </xacro:magnet_plugin_macro>
+  <xacro:magnet_plugin_macro
     namespace="${namespace}"
     suffix="10_left_back_backward"
-    strength="0 0 0.4"
+    strength="0 0 1"
     should_publish="true"
     >
@@ -248,13 +296,13 @@
     namespace="${namespace}"
     suffix="11_left_back_backward"
-    strength="0 0 0.4"
+    strength="0 0 1"
     should_publish="true"
     >
     <origin xyz="-0.135 0.278 0.049" rpy="0 0 1.57079632679" />
-  </xacro:magnet_plugin_macro-->
+  </xacro:magnet_plugin_macro>
   <xacro:magnet_plugin_macro
     namespace="${namespace}"
     suffix="12_left_back_backward"
-    strength="0 0 0.4"
+    strength="0 0 1"
     should_publish="true"
     >

File: big_modquad/config/rotors_description/urdf/multirotor_base.xacro (robot description, xacro)
@@ -147,5 +147,5 @@
       <collision>
         <geometry>
-          <cylinder length="0.005" radius="${radius_rotor}" /> <!-- [m] -->
+          <cylinder length="0.005" radius="${radius_rotor/3}" /> <!-- [m] -->
         </geometry>
       </collision>
